File: Electrical/mcu.kicad_sch (KiCad schematic)
At the start: 6 parts, among them U2 STM32F030F4Px

Commit message: Think I got everything initialized.
Parts:
- added J1, J2: Conn_01x02_MountingPin, symbol Connector_Generic_MountingPin:Conn_01x02_MountingPin
- added SW1: NRST, symbol Switch:SW_Push
- added SW2: BOOT, symbol Switch:SW_Push
Connections:
- net SYS_SWCLK: now also J1.2 (Pin_2)
- net SYS_SWDIO: now also J1.1 (Pin_1)
- net USART1_RX: now also J2.1 (Pin_1)
- net USART1_TX: now also J2.2 (Pin_2)
- net at U2.1 (BOOT0): now also SW2.2
- net at U2.4 (NRST): now also SW1.2
Changed lines of the file:
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@@
   (junction (at 40.64 163.83) (diameter 0) (color 0 0 0 0)
   )
+  (wire (pts (xy 113.03 82.55) (xy 115.57 82.55))
+    (stroke (width 0) (type default))
+  )
   (wire (pts (xy 156.21 71.12) (xy 156.21 81.28))
     (stroke (width 0) (type default))
@@
     (stroke (width 0) (type default))
   )
+  (wire (pts (xy 115.57 82.55) (xy 115.57 86.36))
+    (stroke (width 0) (type default))
+  )
   (wire (pts (xy 198.12 101.6) (xy 168.91 101.6))
     (stroke (width 0) (type default))
@@
     (stroke (width 0) (type default))
   )
+  (wire (pts (xy 250.19 58.42) (xy 251.46 58.42))
+    (stroke (width 0) (type default))
+  )
   (wire (pts (xy 130.81 99.06) (xy 143.51 99.06))
     (stroke (width 0) (type default))
   )
+  (wire (pts (xy 115.57 86.36) (xy 143.51 86.36))
+    (stroke (width 0) (type default))
+  )
   (wire (pts (xy 36.83 186.69) (xy 41.91 186.69))
     (stroke (width 0) (type default))
@@
     (stroke (width 0) (type default))
   )
-  (wire (pts (xy 198.12 114.3) (xy 168.91 114.3))
+  (wire (pts (xy 113.03 91.44) (xy 143.51 91.44))
+    (stroke (width 0) (type default))
+  )
+  (wire (pts (xy 241.3 62.23) (xy 250.19 62.23))
+    (stroke (width 0) (type default))
+  )
+  (wire (pts (xy 168.91 114.3) (xy 199.39 114.3))
     (stroke (width 0) (type default))
   )
@@
     (stroke (width 0) (type default))
   )
-  (wire (pts (xy 198.12 111.76) (xy 168.91 111.76))
-    (stroke (width 0) (type default))
-  )
-  (wire (pts (xy 198.12 93.98) (xy 168.91 93.98))
+  (wire (pts (xy 168.91 111.76) (xy 201.93 111.76))
+    (stroke (width 0) (type default))
+  )
+  (wire (pts (xy 214.63 93.98) (xy 168.91 93.98))
     (stroke (width 0) (type default))
   )
@@
     (stroke (width 0) (type default))
   )
+  (wire (pts (xy 240.03 55.88) (xy 251.46 55.88))
+    (stroke (width 0) (type default))
+  )
   (wire (pts (xy 151.13 71.12) (xy 156.21 71.12))
     (stroke (width 0) (type default))
   )
+  (wire (pts (xy 250.19 62.23) (xy 250.19 58.42))
+    (stroke (width 0) (type default))
+  )
   (wire (pts (xy 198.12 109.22) (xy 168.91 109.22))
     (stroke (width 0) (type default))
   )
-  (wire (pts (xy 198.12 106.68) (xy 168.91 106.68))
+  (wire (pts (xy 199.39 114.3) (xy 199.39 119.38))
+    (stroke (width 0) (type default))
+  )
+  (wire (pts (xy 201.93 111.76) (xy 201.93 119.38))
+    (stroke (width 0) (type default))
+  )
+  (wire (pts (xy 214.63 106.68) (xy 168.91 106.68))
     (stroke (width 0) (type default))
   )
@@
     (effects (font (size 5 5)) (justify left bottom))
   )
+  (label "SYS_SWCLK" (at 199.39 118.11 180) (fields_autoplaced)
+    (effects (font (size 1.27 1.27)) (justify right bottom))
+  )
+  (label "SYS_SWDIO" (at 201.93 114.3 0) (fields_autoplaced)
+    (effects (font (size 1.27 1.27)) (justify left bottom))
+  )
   (label "VDDA" (at 45.72 156.21 0) (fields_autoplaced)
     (effects (font (size 1.27 1.27)) (justify left bottom))
@@
     (effects (font (size 1.27 1.27)) (justify left bottom))
   )
+  (label "USART1_RX" (at 214.63 93.98 0) (fields_autoplaced)
+    (effects (font (size 1.27 1.27)) (justify left bottom))
+  )
+  (label "USART1_RX" (at 240.03 55.88 180) (fields_autoplaced)
+    (effects (font (size 1.27 1.27)) (justify right bottom))
+  )
+  (label "USART1_TX" (at 241.3 62.23 180) (fields_autoplaced)
+    (effects (font (size 1.27 1.27)) (justify right bottom))
+  )
   (label "VDD" (at 54.61 179.07 0) (fields_autoplaced)
+    (effects (font (size 1.27 1.27)) (justify left bottom))
+  )
+  (label "USART1_TX" (at 214.63 106.68 0) (fields_autoplaced)
     (effects (font (size 1.27 1.27)) (justify left bottom))
   )
@@
     (effects (font (size 1.27 1.27)) (justify right))
   )
-  (hierarchical_label "SYS_SWDIO" (shape input) (at 198.12 111.76 0) (fields_autoplaced)
-    (effects (font (size 1.27 1.27)) (justify left))
-  )
-  (hierarchical_label "USART1_TX" (shape input) (at 198.12 106.68 0) (fields_autoplaced)
-    (effects (font (size 1.27 1.27)) (justify left))
-  )
   (hierarchical_label "GPIO_OUTPUT_1" (shape input) (at 198.12 104.14 0) (fields_autoplaced)
     (effects (font (size 1.27 1.27)) (justify left))
@@
     (effects (font (size 1.27 1.27)) (justify left))
   )
-  (hierarchical_label "USART1_RX" (shape input) (at 198.12 93.98 0) (fields_autoplaced)
-    (effects (font (size 1.27 1.27)) (justify left))
-  )
   (hierarchical_label "GPIO_INPUT_3" (shape input) (at 198.12 96.52 0) (fields_autoplaced)
     (effects (font (size 1.27 1.27)) (justify left))
@@
   )
   (hierarchical_label "GPIO_INPUT_0" (shape input) (at 198.12 109.22 0) (fields_autoplaced)
-    (effects (font (size 1.27 1.27)) (justify left))
-  )
-  (hierarchical_label "SYS_SWCLK" (shape input) (at 198.12 114.3 0) (fields_autoplaced)
     (effects (font (size 1.27 1.27)) (justify left))
   )
@@
     )
   )
+  (symbol (lib_id "Connector_Generic_MountingPin:Conn_01x02_MountingPin") (at 201.93 124.46 270) (unit 1)
+    (in_bom yes) (on_board yes) (dnp no)
+    (property "Reference" "J1" (at 204.47 123.19 90)
+      (effects (font (size 1.27 1.27)) (justify left))
+    )
+    (property "Value" "Conn_01x02_MountingPin" (at 190.5 125.73 90)
+      (effects (font (size 1.27 1.27)) (justify left))
+    )
+    (property "Footprint" "" (at 201.93 124.46 0)
+      (effects (font (size 1.27 1.27)) hide)
+    )
+    (property "Datasheet" "~" (at 201.93 124.46 0)
+      (effects (font (size 1.27 1.27)) hide)
+    )
+    (pin "1")
+    (pin "2")
+    (pin "MP")
+    (instances
+      (project "Electrical"
+        (path "/869aa179-d08c-47d1-91ac-ef955a1d76ce/96565827-501d-4f65-a2e2-c37deaebcaa3"
+          (reference "J1") (unit 1)
+        )
+      )
+    )
+  )
   (symbol (lib_id "Device:C") (at 33.02 160.02 0) (unit 1)
     (in_bom yes) (on_board yes) (dnp no) (fields_autoplaced)
@@
     )
   )
+  (symbol (lib_id "Connector_Generic_MountingPin:Conn_01x02_MountingPin") (at 256.54 55.88 0) (unit 1)
+    (in_bom yes) (on_board yes) (dnp no)
+    (property "Reference" "J2" (at 255.27 53.34 90)
+      (effects (font (size 1.27 1.27)) (justify left))
+    )
+    (property "Value" "Conn_01x02_MountingPin" (at 257.81 67.31 90)
+      (effects (font (size 1.27 1.27)) (justify left))
+    )
+    (property "Footprint" "" (at 256.54 55.88 0)
+      (effects (font (size 1.27 1.27)) hide)
+    )
+    (property "Datasheet" "~" (at 256.54 55.88 0)
+      (effects (font (size 1.27 1.27)) hide)
+    )
+    (pin "1")
+    (pin "2")
+    (pin "MP")
+    (instances
+      (project "Electrical"
+        (path "/869aa179-d08c-47d1-91ac-ef955a1d76ce/96565827-501d-4f65-a2e2-c37deaebcaa3"
+          (reference "J2") (unit 1)
+        )
+      )
+    )
+  )
+  (symbol (lib_id "Switch:SW_Push") (at 107.95 91.44 0) (unit 1)
+    (in_bom yes) (on_board yes) (dnp no)
+    (property "Reference" "SW2" (at 107.95 87.63 0)
+      (effects (font (size 1.27 1.27)))
+    )
+    (property "Value" "BOOT" (at 107.95 92.71 0)
+      (effects (font (size 1.27 1.27)))
+    )
+    (property "Footprint" "" (at 107.95 86.36 0)
+      (effects (font (size 1.27 1.27)) hide)
+    )
+    (property "Datasheet" "~" (at 107.95 86.36 0)
+      (effects (font (size 1.27 1.27)) hide)
+    )
+    (pin "1")
+    (pin "2")
+    (instances
+      (project "Electrical"
+        (path "/869aa179-d08c-47d1-91ac-ef955a1d76ce/96565827-501d-4f65-a2e2-c37deaebcaa3"
+          (reference "SW2") (unit 1)
+        )
+      )
+    )
+  )
   (symbol (lib_id "power:+3.3V") (at 33.02 156.21 0) (unit 1)
     (in_bom yes) (on_board yes) (dnp no) (fields_autoplaced)
@@
         )
       )
+    )
+  )
+  (symbol (lib_id "Switch:SW_Push") (at 107.95 82.55 0) (unit 1)
+    (in_bom yes) (on_board yes) (dnp no) (fields_autoplaced)
+    (property "Reference" "SW1" (at 107.95 74.93 0)
+      (effects (font (size 1.27 1.27)))
+    )
+    (property "Value" "NRST" (at 107.95 77.47 0)
+      (effects (font (size 1.27 1.27)))
+    )
+    (property "Footprint" "" (at 107.95 77.47 0)
+      (effects (font (size 1.27 1.27)) hide)
+    )
+    (property "Datasheet" "~" (at 107.95 77.47 0)
+      (effects (font (size 1.27 1.27)) hide)
+    )
+    (pin "1")
+    (pin "2")
+    (instances
+      (project "Electrical"
+        (path "/869aa179-d08c-47d1-91ac-ef955a1d76ce/96565827-501d-4f65-a2e2-c37deaebcaa3"
+          (reference "SW1") (unit 1)
+        )
+      )

Commit message: Working on it
Parts:
- added C8: 0.1u, symbol Device:C
Connections:
- net +3.3V: now also SW2.1
- net GND: now also SW1.1, C8.1
- net at SW1.2, U2.4 (NRST): now also C8.2
Changed lines of the file:
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@@
 (kicad_sch (version 20230121) (generator eeschema)
   (paper "A4")
+  (junction (at 124.46 86.36) (diameter 0) (color 0 0 0 0)
+  )
   (junction (at 41.91 186.69) (diameter 0) (color 0 0 0 0)
   )
@@
     (stroke (width 0) (type default))
   )
-  (wire (pts (xy 115.57 86.36) (xy 143.51 86.36))
+  (wire (pts (xy 115.57 86.36) (xy 124.46 86.36))
     (stroke (width 0) (type default))
   )
@@
   )
   (wire (pts (xy 40.64 163.83) (xy 45.72 163.83))
+    (stroke (width 0) (type default))
+  )
+  (wire (pts (xy 124.46 86.36) (xy 143.51 86.36))
     (stroke (width 0) (type default))
   )
@@
     )
   )
+  (symbol (lib_id "power:GND") (at 124.46 78.74 180) (unit 1)
+    (in_bom yes) (on_board yes) (dnp no) (fields_autoplaced)
+    (property "Reference" "#PWR011" (at 124.46 72.39 0)
+      (effects (font (size 1.27 1.27)) hide)
+    )
+    (property "Value" "GND" (at 124.46 73.66 0)
+      (effects (font (size 1.27 1.27)))
+    )
+    (property "Footprint" "" (at 124.46 78.74 0)
+      (effects (font (size 1.27 1.27)) hide)
+    )
+    (property "Datasheet" "" (at 124.46 78.74 0)
+      (effects (font (size 1.27 1.27)) hide)
+    )
+    (pin "1")
+    (instances
+      (project "Electrical"
+        (path "/869aa179-d08c-47d1-91ac-ef955a1d76ce/96565827-501d-4f65-a2e2-c37deaebcaa3"
+          (reference "#PWR011") (unit 1)
+        )
+      )
+    )
+  )
   (symbol (lib_id "Device:C") (at 29.21 182.88 0) (unit 1)
     (in_bom yes) (on_board yes) (dnp no) (fields_autoplaced)
@@
     )
   )
+  (symbol (lib_id "power:+3.3V") (at 102.87 91.44 90) (unit 1)
+    (in_bom yes) (on_board yes) (dnp no) (fields_autoplaced)
+    (property "Reference" "#PWR012" (at 106.68 91.44 0)
+      (effects (font (size 1.27 1.27)) hide)
+    )
+    (property "Value" "+3.3V" (at 99.06 91.44 90)
+      (effects (font (size 1.27 1.27)) (justify left))
+    )
+    (property "Footprint" "" (at 102.87 91.44 0)
+      (effects (font (size 1.27 1.27)) hide)
+    )
+    (property "Datasheet" "" (at 102.87 91.44 0)
+      (effects (font (size 1.27 1.27)) hide)
+    )
+    (pin "1")
+    (instances
+      (project "Electrical"
+        (path "/869aa179-d08c-47d1-91ac-ef955a1d76ce/96565827-501d-4f65-a2e2-c37deaebcaa3"
+          (reference "#PWR012") (unit 1)
+        )
+      )
+    )
+  )
+  (symbol (lib_id "power:GND") (at 102.87 82.55 270) (unit 1)
+    (in_bom yes) (on_board yes) (dnp no) (fields_autoplaced)
+    (property "Reference" "#PWR08" (at 96.52 82.55 0)
+      (effects (font (size 1.27 1.27)) hide)
+    )
+    (property "Value" "GND" (at 99.06 82.55 90)
+      (effects (font (size 1.27 1.27)) (justify right))
+    )
+    (property "Footprint" "" (at 102.87 82.55 0)
+      (effects (font (size 1.27 1.27)) hide)
+    )
+    (property "Datasheet" "" (at 102.87 82.55 0)
+      (effects (font (size 1.27 1.27)) hide)
+    )
+    (pin "1")
+    (instances
+      (project "Electrical"
+        (path "/869aa179-d08c-47d1-91ac-ef955a1d76ce/96565827-501d-4f65-a2e2-c37deaebcaa3"
+          (reference "#PWR08") (unit 1)
+        )
+      )
+    )
+  )
   (symbol (lib_id "Switch:SW_Push") (at 107.95 82.55 0) (unit 1)
     (in_bom yes) (on_board yes) (dnp no) (fields_autoplaced)
@@
         )
       )
+    )
+  )
+  (symbol (lib_id "Device:C") (at 124.46 82.55 0) (unit 1)
+    (in_bom yes) (on_board yes) (dnp no) (fields_autoplaced)
+    (property "Reference" "C8" (at 128.27 81.28 0)
+      (effects (font (size 1.27 1.27)) (justify left))
+    )
+    (property "Value" "0.1u" (at 128.27 83.82 0)
+      (effects (font (size 1.27 1.27)) (justify left))
+    )
+    (property "Footprint" "" (at 125.4252 86.36 0)
+      (effects (font (size 1.27 1.27)) hide)
+    )
+    (property "Datasheet" "~" (at 124.46 82.55 0)
+      (effects (font (size 1.27 1.27)) hide)
+    )
+    (pin "1")
+    (pin "2")
+    (instances
+      (project "Electrical"
+        (path "/869aa179-d08c-47d1-91ac-ef955a1d76ce/96565827-501d-4f65-a2e2-c37deaebcaa3"
+          (reference "C8") (unit 1)
+        )
+      )
