File: Electrical/Electrical.kicad_sch (KiCad schematic)
At the start: 6 parts, among them M1 Fan, M2 Fan, M3 Fan, M4 Fan, M5 Fan

Commit message: Working on schematic
Other:
- added sheet MCU (mcu.kicad_sch)
Changed lines of the file:
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@@
       (effects (font (size 1.27 1.27)) hide)
     )
+    (pin "1")
     (pin "2")
-    (pin "1")
     (instances
       (project "Electrical"
@@
       (effects (font (size 1.27 1.27)) hide)
     )
+    (pin "1")
     (pin "2")
-    (pin "1")
     (instances
       (project "Electrical"
@@
       (effects (font (size 1.27 1.27)) hide)
     )
+    (pin "1")
     (pin "2")
-    (pin "1")
     (instances
       (project "Electrical"
@@
       (effects (font (size 1.27 1.27)) hide)
     )
+    (pin "1")
     (pin "2")
-    (pin "1")
     (instances
       (project "Electrical"
@@
       (effects (font (size 1.27 1.27)) hide)
     )
+    (pin "1")
     (pin "2")
-    (pin "1")
     (instances
       (project "Electrical"
@@
     )
   )
-  (sheet (at 207.01 41.91) (size 27.94 21.59) (fields_autoplaced)
+  (sheet (at 219.71 69.85) (size 27.94 21.59) (fields_autoplaced)
     (stroke (width 0.1524) (type solid))
     (fill (color 0 0 0 0.0000))
-    (property "Sheetname" "tmpPhy" (at 207.01 41.1984 0)
+    (property "Sheetname" "tmpPhy" (at 219.71 69.1384 0)
       (effects (font (size 1.27 1.27)) (justify left bottom))
     )
-    (property "Sheetfile" "tempphy.kicad_sch" (at 207.01 64.0846 0)
+    (property "Sheetfile" "tempphy.kicad_sch" (at 219.71 92.0246 0)
       (effects (font (size 1.27 1.27)) (justify left top))
     )
-    (pin "MTRCTRL1" input (at 207.01 50.8 180)
+    (pin "MTRCTRL1" input (at 219.71 78.74 180)
       (effects (font (size 1.27 1.27)) (justify left))
     )
-    (pin "MTRCTRL2" input (at 207.01 54.61 180)
+    (pin "MTRCTRL2" input (at 219.71 82.55 180)
       (effects (font (size 1.27 1.27)) (justify left))
     )
@@
       )
     )
+  )
+  (sheet (at 81.28 106.68) (size 25.4 16.51) (fields_autoplaced)
+    (stroke (width 0.1524) (type solid))
+    (fill (color 0 0 0 0.0000))
+    (property "Sheetname" "MCU" (at 81.28 105.9684 0)
+      (effects (font (size 1.27 1.27)) (justify left bottom))
+    )
+    (property "Sheetfile" "mcu.kicad_sch" (at 81.28 123.7746 0)
+      (effects (font (size 1.27 1.27)) (justify left top))
+    )
+    (instances
+      (project "Electrical"
+        (path "/869aa179-d08c-47d1-91ac-ef955a1d76ce" (page "3"))
+      )
+    )

Commit message: Working on it
Parts:
- removed M3, M4, M5: Fan, symbol Motor:Fan
- added A1: Arduino_UNO_R3, Module:Arduino_UNO_R3, symbol MCU_Module:Arduino_UNO_R3
- added J1: DISPLAY, symbol Connector:Conn_01x04_Pin
- added M6, M7, M8: Fan, Connector_PinHeader_2.54mm:PinHeader_1x02_P2.54mm_Vertical, symbol Motor:Fan
- added Q1, Q2: NMOS, symbol Simulation_SPICE:NMOS
- added R2, R3: 10k, symbol Device:R
- added SW1: RotaryEncoder_Switch, symbol Device:RotaryEncoder_Switch
- added TH2, TH3: 3950b-10k, Connector_PinHeader_2.54mm:PinHeader_1x02_P2.54mm_Vertical, symbol Device:Thermistor
- M1, M2, TH1: footprint (none) -> Connector_PinHeader_2.54mm:PinHeader_1x02_P2.54mm_Vertical
Connections:
- net +5V: now also A1.5 (+5V), SW1.C, SW1.S1; no longer TH1.1
- net tmpPhy/MTRCTRL1: now also A1.18 (D3)
- net tmpPhy/MTRCTRL2: now also A1.19 (D4)
- net +12V: now reaches M2.1 (+)
- net +12V: now also M1.1 (+), A1.8 (VIN), M6.1 (+), M7.1 (+), M8.1 (+)
- net at M2.2 (-): now also M1.2 (-), Q1.1 (D)
- net at TH1.2: now also A1.9 (A0)
- new net: A1.30 (AREF), TH1.1, TH2.1, TH3.1
- new net: A1.11 (A2), TH3.2
- new net: M6.2 (-), M7.2 (-), M8.2 (-), Q2.1 (D)
- new net: A1.10 (A1), TH2.2
- new net +3.3V: A1.4 (3V3), J1.3 (Pin_3)
- new net GND: A1.29 (GND), A1.6 (GND), A1.7 (GND), J1.4 (Pin_4), Q1.3 (S), Q2.3 (S), R2.2, R3.2
- new net INSIDE_CTRL: A1.17 (D2), Q1.2 (G), R2.1
- new net OUTSIDE_CTRL: A1.20 (D5), Q2.2 (G), R3.1
- new net RTRY_A: A1.22 (D7), SW1.A
- new net RTRY_B: A1.23 (D8), SW1.B
- new net RTRY_SW: A1.21 (D6), SW1.S2
- new net SCL: A1.32 (SCL/A5), J1.2 (Pin_2)
- new net SDA: A1.31 (SDA/A4), J1.1 (Pin_1)
Other:
- removed sheet MCU
- moved on the sheet: M2, TH1

Commit message: Finished with Schematic and BOM.
Parts:
- removed SW1: RotaryEncoder_Switch, symbol Device:RotaryEncoder_Switch
- added SW1, SW3: GT-TC149A-H060-L1, TTC:KEY-SMD_4P-L12.0-W12.0-P5.00-LS15.2, symbol TTC:GT-TC149A-H060-L1
- added SW2: EC111012000Y, TTC:SW-TH_EC111012000Y, symbol TTC:EC111012000Y
- J1, M1, M2, M6, M7, M8, TH1, TH2, TH3: LCSC_ID (none) -> NOPOP
- Q1, Q2: footprint (none) -> Package_DFN_QFN:WDFN-8-1EP_4x3mm_P0.65mm_EP2.4x1.8mm_ThermalVias; LCSC_ID (none) -> C893914
- R2, R3: footprint (none) -> Resistor_SMD:R_0402_1005Metric; LCSC_ID (none) -> C60490
Connections:
- net +5V: now also SW1.1, SW2.C, SW3.1
- net RTRY_A: now also SW2.A
- net RTRY_B: now also SW2.B
- net at A1.24 (D9): now also SW3.4
- net RTRY_SW: no longer names the net of A1.21 (D6)
- net RTRY_SW: now also SW1.4
