File: Electrical/tempphy.kicad_sch (KiCad schematic)
At the start: 6 parts

Commit message: Working on schematic
Changed lines of the file:
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@@
       (effects (font (size 1.27 1.27)) hide)
     )
+    (pin "1")
     (pin "2")
-    (pin "1")
     (instances
       (project "Electrical"
@@
     )
     (pin "1")
-    (pin "7")
-    (pin "6")
-    (pin "5")
+    (pin "2")
     (pin "3")
     (pin "4")
-    (pin "2")
+    (pin "5")
+    (pin "6")
+    (pin "7")
+    (pin "8")
     (pin "9")
-    (pin "8")
     (instances
       (project "Electrical"
@@
     )
     (property "Value" "GND" (at 118.11 104.14 0)
-      (effects (font (size 1.27 1.27)))
+      (effects (font (size 1.27 1.27)) hide)
     )
     (property "Footprint" "" (at 118.11 99.06 0)

Commit message: Working on it
Parts:
- C?: value 0.1u -> 100n; footprint (none) -> Capacitor_SMD:C_0402_1005Metric; LCSC_ID (none) -> C56392
- PE? (x2): footprint (none) -> Connector_PinHeader_2.54mm:PinHeader_1x02_P2.54mm_Vertical
Changed lines of the file:
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@@
+      (effects (font (size 1.27 1.27)) hide)
+    )
+    (property "LCSC_ID" "" (at 125.73 54.61 0)
       (effects (font (size 1.27 1.27)) hide)
     )
@@
       (effects (font (size 1.27 1.27)) (justify left))
     )
-    (property "Footprint" "" (at 140.462 85.09 0)
+    (property "Footprint" "Connector_PinHeader_2.54mm:PinHeader_1x02_P2.54mm_Vertical" (at 140.462 85.09 0)
       (effects (font (size 1.27 1.27)) hide)
     )
     (property "Datasheet" "~" (at 142.875 85.09 90)
+      (effects (font (size 1.27 1.27)) hide)
+    )
+    (property "LCSC_ID" "" (at 142.24 85.09 0)
       (effects (font (size 1.27 1.27)) hide)
     )
@@
       (effects (font (size 1.27 1.27)) hide)
     )
+    (property "LCSC_ID" "" (at 138.43 97.79 0)
+      (effects (font (size 1.27 1.27)) hide)
+    )
     (pin "1")
     (pin "2")
@@
       (effects (font (size 1.27 1.27)) (justify left))
     )
-    (property "Value" "0.1u" (at 127 72.39 90)
+    (property "Value" "100n" (at 127 72.39 90)
       (effects (font (size 1.27 1.27)) (justify left))
     )
-    (property "Footprint" "" (at 129.54 67.6148 0)
+    (property "Footprint" "Capacitor_SMD:C_0402_1005Metric" (at 129.54 67.6148 0)
       (effects (font (size 1.27 1.27)) hide)
     )
     (property "Datasheet" "~" (at 125.73 68.58 0)
+      (effects (font (size 1.27 1.27)) hide)
+    )
+    (property "LCSC_ID" "C56392" (at 125.73 68.58 0)
       (effects (font (size 1.27 1.27)) hide)
     )
@@
       (effects (font (size 1.27 1.27)) (justify left))
     )
-    (property "Footprint" "" (at 162.052 85.09 0)
+    (property "Footprint" "Connector_PinHeader_2.54mm:PinHeader_1x02_P2.54mm_Vertical" (at 162.052 85.09 0)
       (effects (font (size 1.27 1.27)) hide)
     )
     (property "Datasheet" "~" (at 164.465 85.09 90)
+      (effects (font (size 1.27 1.27)) hide)
+    )
+    (property "LCSC_ID" "" (at 163.83 85.09 0)
       (effects (font (size 1.27 1.27)) hide)
     )
@@
       (effects (font (size 1.27 1.27)) hide)
     )
+    (property "LCSC_ID" "" (at 118.11 87.63 0)
+      (effects (font (size 1.27 1.27)) hide)
+    )

Commit message: Finished with Schematic and BOM.
Parts:
- C?: footprint (none) -> Capacitor_Tantalum_SMD:CP_EIA-3528-21_Kemet-B; LCSC_ID (none) -> C136751
- PE? (x2): LCSC_ID (none) -> NOPOP
- R1: footprint (none) -> Resistor_SMD:R_0402_1005Metric; LCSC_ID (none) -> C25756
- U?: LCSC_ID (none) -> C75864
Changed lines of the file:
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@@
       (effects (font (size 1.27 1.27)))
     )
-    (property "Footprint" "" (at 129.54 53.6448 0)
+    (property "Footprint" "Capacitor_Tantalum_SMD:CP_EIA-3528-21_Kemet-B" (at 129.54 53.6448 0)
       (effects (font (size 1.27 1.27)) hide)
     )
@@
       (effects (font (size 1.27 1.27)) hide)
     )
-    (property "LCSC_ID" "" (at 125.73 54.61 0)
+    (property "LCSC_ID" "C136751" (at 125.73 54.61 0)
       (effects (font (size 1.27 1.27)) hide)
     )
@@
       (effects (font (size 1.27 1.27)) hide)
     )
-    (property "LCSC_ID" "" (at 142.24 85.09 0)
+    (property "LCSC_ID" "NOPOP" (at 142.24 85.09 0)
       (effects (font (size 1.27 1.27)) hide)
     )
@@
       (effects (font (size 1.27 1.27)) (justify left))
     )
-    (property "Footprint" "" (at 136.652 97.79 90)
+    (property "Footprint" "Resistor_SMD:R_0402_1005Metric" (at 136.652 97.79 90)
       (effects (font (size 1.27 1.27)) hide)
     )
@@
       (effects (font (size 1.27 1.27)) hide)
     )
-    (property "LCSC_ID" "" (at 138.43 97.79 0)
+    (property "LCSC_ID" "C25756" (at 138.43 97.79 0)
       (effects (font (size 1.27 1.27)) hide)
     )
@@
       (effects (font (size 1.27 1.27)) hide)
     )
-    (property "LCSC_ID" "" (at 163.83 85.09 0)
+    (property "LCSC_ID" "NOPOP" (at 163.83 85.09 0)
       (effects (font (size 1.27 1.27)) hide)
     )
@@
       (effects (font (size 1.27 1.27)) hide)
     )
-    (property "LCSC_ID" "" (at 118.11 87.63 0)
+    (property "LCSC_ID" "C75864" (at 118.11 87.63 0)
       (effects (font (size 1.27 1.27)) hide)
     )
